File: USB_DAC-AMP_WITH_TONE_CTRL/USB_DAC-AMP_WITH_TONE_CTRL.kicad_sch (KiCad schematic)
At the start: 121 parts, among them J1 USB_C_Receptacle, J2 SJ-3524-SMT, SW1 SW_Push, U1 PCM2906, U10 NE5532, U11 NE5532, U2 TPS61040DBV, U3 SPX3819M5-L, U4 SPX3819M5-L, U5 NE5532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

Commit message: finished USB_DAC-AMP schematic
Parts:
- removed C37: 100u, Capacitor_Tantalum_SMD:CP_EIA-7343-15_Kemet-W, symbol Device:C
- removed C38, C42, C44: 100n, symbol Device:C
- removed C39: 2.2n, symbol Device:C
- removed C40, C41: 100u, symbol Device:C
- removed C43, C46: 30p, symbol Device:C
- removed C45: 1000u, symbol Device:C
- removed D7: D_TVS, symbol Device:D_TVS
- removed FB5: 120R, symbol Device:FerriteBead
- removed J2: SJ-3524-SMT, SJ-3524-SMT:CUI_SJ-3524-SMT, symbol Imported_symbols:SJ-3524-SMT
- removed R34, R39: 22K, symbol Device:R
- removed R35, R36, R38, R43: 1.5K, symbol Device:R
- removed R40: 5.1K, symbol Device:R
- removed R41, R42: 1, symbol Device:R
- removed U11: NE5532, symbol Amplifier_Operational:NE5532
- removed unit 2 of U6
- added J3: AudioJack3, symbol Connector_Audio:AudioJack3
- added R4: PTN092-H20115K1A, PTN092-H20115K1A:TRIM_PTN092-H20115K1A, symbol PTN092-H20115K1A:PTN092-H20115K1A
- C25: footprint Capacitor_Tantalum_SMD:CP_EIA-7343-15_Kemet-W -> (none)
Connections:
- net +15VA: no longer U10.8 (V+), U8.8 (V+)
- net GND: no longer U10.4 (V-), U8.4 (V-)
- net VBL: no longer U6.1, U6.2 (-)
- net at U10.7: no longer R3.3_2
- net at U10.1: no longer U10.2 (-)
- net at U8.1: no longer U8.2 (-)
- net at C36.2, D6.2 (A2), FB4.2: now also J3.T
- net at U8.6 (-): no longer U8.7
- net at R3.1_1: no longer C30.2
- new net MID: U6.1, U6.2 (-)
- no-connect marks 15 -> 14
Other:
- note removed: "Electrolytic, fairly large, feeding into buffer"
- moved on the sheet: C25, C26, C27, C28, C29, C30, C31, C32, C33, C34, C35, C36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
