File: USB_DAC-AMP/USB_DAC-AMP.kicad_pcb (KiCad board)
At the start: 2 copper layers, 9 parts, among them J2 SJ-3524-SMT, U1 PCM2906, U2 TPS61040DBV, U3 SPX3819M5-L, U4 SPX3819M5-L

Commit message: finished V1 footprint assignments
Parts:
- removed R4: PTN092-H20115K1A, PTN092-H20115K1A:TRIM_PTN092-H20115K1A
- added C1: 10u, Capacitor_SMD:C_0603_1608Metric_Pad1.08x0.95mm_HandSolder, F.Cu at (106.3, 88.0)
- added C10: 10u, Capacitor_SMD:C_0603_1608Metric_Pad1.08x0.95mm_HandSolder, F.Cu at (245.6, 47.3)
- added C11: 10u, Capacitor_SMD:C_0603_1608Metric_Pad1.08x0.95mm_HandSolder, F.Cu at (250.0, 24.7)
- added C12: 10u, Capacitor_SMD:C_0603_1608Metric_Pad1.08x0.95mm_HandSolder, F.Cu at (138.3, 49.4)
- added C13: 10u, Capacitor_SMD:C_0603_1608Metric_Pad1.08x0.95mm_HandSolder, F.Cu at (144.1, 49.4)
- added C14: 1000u, Capacitor_Tantalum_SMD:CP_EIA-7343-43_Kemet-X_HandSolder, F.Cu at (228.0, 26.3)
- added C15: 1000u, Capacitor_Tantalum_SMD:CP_EIA-7343-43_Kemet-X_HandSolder, F.Cu at (228.0, 32.2)
- added C16: 1u, Capacitor_SMD:C_0603_1608Metric_Pad1.08x0.95mm_HandSolder, F.Cu at (250.0, 32.2)
- added C17: 1u, Capacitor_SMD:C_0603_1608Metric_Pad1.08x0.95mm_HandSolder, F.Cu at (250.0, 34.7)
- added C18: 1u, Capacitor_SMD:C_0603_1608Metric_Pad1.08x0.95mm_HandSolder, F.Cu at (250.0, 37.2)
- added C19: 10u, Capacitor_SMD:C_0603_1608Metric_Pad1.08x0.95mm_HandSolder, F.Cu at (250.0, 39.7)
- added C2: 30p, Capacitor_SMD:C_0603_1608Metric_Pad1.08x0.95mm_HandSolder, F.Cu at (245.6, 27.2)
- added C20: 1u, Capacitor_SMD:C_0603_1608Metric_Pad1.08x0.95mm_HandSolder, F.Cu at (250.0, 42.2)
- added C21: 1u, Capacitor_SMD:C_0603_1608Metric_Pad1.08x0.95mm_HandSolder, F.Cu at (250.0, 44.8)
- added C22: 1u, Capacitor_SMD:C_0603_1608Metric_Pad1.08x0.95mm_HandSolder, F.Cu at (250.0, 47.3)
- added C23: 30p, Capacitor_SMD:C_0603_1608Metric_Pad1.08x0.95mm_HandSolder, F.Cu at (254.3, 24.7)
- added C24: 30p, Capacitor_SMD:C_0603_1608Metric_Pad1.08x0.95mm_HandSolder, F.Cu at (254.3, 27.2)
- added C25: 100u, Capacitor_Tantalum_SMD:CP_EIA-7343-43_Kemet-X_HandSolder, F.Cu at (228.0, 38.0)
- added C26: 100n, Capacitor_SMD:C_0603_1608Metric_Pad1.08x0.95mm_HandSolder, F.Cu at (254.3, 29.7)
- added C27: 1000u, Capacitor_Tantalum_SMD:CP_EIA-7343-43_Kemet-X_HandSolder, F.Cu at (228.0, 43.9)
- added C28: 100n, Capacitor_SMD:C_0603_1608Metric_Pad1.08x0.95mm_HandSolder, F.Cu at (254.3, 32.2)
- added C29: 2.2n, Capacitor_SMD:C_0603_1608Metric_Pad1.08x0.95mm_HandSolder, F.Cu at (254.3, 34.7)
- added C3: 30p, Capacitor_SMD:C_0603_1608Metric_Pad1.08x0.95mm_HandSolder, F.Cu at (245.6, 29.7)
- added C30: 100u, Capacitor_Tantalum_SMD:CP_EIA-7343-43_Kemet-X_HandSolder, F.Cu at (228.0, 49.7)
- added C31: 100u, Capacitor_Tantalum_SMD:CP_EIA-7343-43_Kemet-X_HandSolder, F.Cu at (228.0, 55.6)
- added C32: 100n, Capacitor_SMD:C_0603_1608Metric_Pad1.08x0.95mm_HandSolder, F.Cu at (254.3, 37.2)
- added C33: 30p, Capacitor_SMD:C_0603_1608Metric_Pad1.08x0.95mm_HandSolder, F.Cu at (254.3, 39.7)
- added C34: 100n, Capacitor_SMD:C_0603_1608Metric_Pad1.08x0.95mm_HandSolder, F.Cu at (254.3, 42.2)
- added C35: 1000u, Capacitor_Tantalum_SMD:CP_EIA-7343-43_Kemet-X_HandSolder, F.Cu at (228.0, 61.4)
- added C36: 30p, Capacitor_SMD:C_0603_1608Metric_Pad1.08x0.95mm_HandSolder, F.Cu at (254.3, 44.8)
- added C37: 100u, Capacitor_Tantalum_SMD:CP_EIA-7343-15_Kemet-W, F.Cu at (248.4, 77.9)
- added C38: 100n, Capacitor_SMD:C_0603_1608Metric_Pad1.08x0.95mm_HandSolder, F.Cu at (254.3, 47.3)
- added C39: 2.2n, Capacitor_SMD:C_0603_1608Metric_Pad1.08x0.95mm_HandSolder, F.Cu at (258.7, 24.7)
- added C4: 30p, Capacitor_SMD:C_0603_1608Metric_Pad1.08x0.95mm_HandSolder, F.Cu at (245.6, 32.2)
- added C40: 100u, Capacitor_Tantalum_SMD:CP_EIA-7343-43_Kemet-X_HandSolder, F.Cu at (228.0, 67.3)
- added C41: 100u, Capacitor_Tantalum_SMD:CP_EIA-7343-43_Kemet-X_HandSolder, F.Cu at (228.0, 73.1)
- added C42: 100n, Capacitor_SMD:C_0603_1608Metric_Pad1.08x0.95mm_HandSolder, F.Cu at (258.7, 27.2)
- added C43: 30p, Capacitor_SMD:C_0603_1608Metric_Pad1.08x0.95mm_HandSolder, F.Cu at (258.7, 29.7)
- added C44: 100n, Capacitor_SMD:C_0603_1608Metric_Pad1.08x0.95mm_HandSolder, F.Cu at (258.7, 32.2)
- added C45: 1000u, Capacitor_Tantalum_SMD:CP_EIA-7343-43_Kemet-X_HandSolder, F.Cu at (228.0, 79.0)
- added C46: 30p, Capacitor_SMD:C_0603_1608Metric_Pad1.08x0.95mm_HandSolder, F.Cu at (258.7, 34.7)
- added C5: 30p, Capacitor_SMD:C_0603_1608Metric_Pad1.08x0.95mm_HandSolder, F.Cu at (245.6, 34.7)
- added C6: 30p, Capacitor_SMD:C_0603_1608Metric_Pad1.08x0.95mm_HandSolder, F.Cu at (110.5, 84.5)
- added C7: 1u, Capacitor_SMD:C_0603_1608Metric_Pad1.08x0.95mm_HandSolder, F.Cu at (245.6, 39.7)
- added C8: 1u, Capacitor_SMD:C_0603_1608Metric_Pad1.08x0.95mm_HandSolder, F.Cu at (245.6, 42.2)
- added C9: 10u, Capacitor_SMD:C_0603_1608Metric_Pad1.08x0.95mm_HandSolder, F.Cu at (124.8, 51.1)
- added D1: D_TVS, Diode_SMD:D_0603_1608Metric_Pad1.05x0.95mm_HandSolder, F.Cu at (269.2, 61.6)
- added D2: 0603ESDA-18N, Diode_SMD:D_0603_1608Metric_Pad1.05x0.95mm_HandSolder, F.Cu at (269.2, 64.2)
- added D3: LED, LED_SMD:LED_0603_1608Metric_Pad1.05x0.95mm_HandSolder, F.Cu at (269.2, 66.7)
- added D6: D_TVS, Diode_SMD:D_0603_1608Metric_Pad1.05x0.95mm_HandSolder, F.Cu at (269.2, 69.3)
- added D7: D_TVS, Diode_SMD:D_0603_1608Metric_Pad1.05x0.95mm_HandSolder, F.Cu at (269.2, 71.9)
- added F1: Polyfuse - 750mA, Fuse:Fuse_0603_1608Metric_Pad1.05x0.95mm_HandSolder, F.Cu at (258.7, 37.2)
- added FB1: 120R, Resistor_SMD:R_0603_1608Metric_Pad0.98x0.95mm_HandSolder, F.Cu at (258.7, 39.7)
- added FB2: 120R, Resistor_SMD:R_0603_1608Metric_Pad0.98x0.95mm_HandSolder, F.Cu at (133.7, 48.5)
- added FB3: 120R, Resistor_SMD:R_0603_1608Metric_Pad0.98x0.95mm_HandSolder, F.Cu at (258.7, 44.8)
- added FB4: 120R, Resistor_SMD:R_0603_1608Metric_Pad0.98x0.95mm_HandSolder, F.Cu at (258.7, 47.3)
- added FB5: 120R, Resistor_SMD:R_0603_1608Metric_Pad0.98x0.95mm_HandSolder, F.Cu at (263.0, 24.7)
- added J1: USB_C_Receptacle, Connector_USB:USB_C_Receptacle_GCT_USB4105-xx-A_16P_TopMnt_Horizontal, F.Cu at (35.4, 87.6)
- added L1: 10u, Inductor_SMD:L_0805_2012Metric_Pad1.05x1.20mm_HandSolder, F.Cu at (109.3, 90.7)
- added R1: 5.1K, Resistor_SMD:R_0603_1608Metric_Pad0.98x0.95mm_HandSolder, F.Cu at (263.0, 27.2)
- added R10: 240K, Resistor_SMD:R_0603_1608Metric_Pad0.98x0.95mm_HandSolder, F.Cu at (143.0, 52.1)
- added R11: 22K, Resistor_SMD:R_0603_1608Metric_Pad0.98x0.95mm_HandSolder, F.Cu at (139.2, 52.1)
- added R12: 20, Resistor_SMD:R_0603_1608Metric_Pad0.98x0.95mm_HandSolder, F.Cu at (267.4, 24.7)
- added R13: 1.5K, Resistor_SMD:R_0603_1608Metric_Pad0.98x0.95mm_HandSolder, F.Cu at (267.4, 27.2)
- added R14: 22, Resistor_SMD:R_0603_1608Metric_Pad0.98x0.95mm_HandSolder, F.Cu at (267.4, 29.7)
- added R15: 22, Resistor_SMD:R_0603_1608Metric_Pad0.98x0.95mm_HandSolder, F.Cu at (267.4, 32.2)
- added R16: 1.5K, Resistor_SMD:R_0603_1608Metric_Pad0.98x0.95mm_HandSolder, F.Cu at (267.4, 34.7)
- added R17: 2.2, Resistor_SMD:R_0603_1608Metric_Pad0.98x0.95mm_HandSolder, F.Cu at (267.4, 37.2)
- added R2: 5.1K, Resistor_SMD:R_0603_1608Metric_Pad0.98x0.95mm_HandSolder, F.Cu at (263.0, 29.7)
- added R20: 1.5k, Resistor_SMD:R_0603_1608Metric_Pad0.98x0.95mm_HandSolder, F.Cu at (267.4, 39.7)
- added R21: 1.5k, Resistor_SMD:R_0603_1608Metric_Pad0.98x0.95mm_HandSolder, F.Cu at (267.4, 42.2)
- added R22: 1M, Resistor_SMD:R_0603_1608Metric_Pad0.98x0.95mm_HandSolder, F.Cu at (267.4, 44.8)
- added R23: 22K, Resistor_SMD:R_0603_1608Metric_Pad0.98x0.95mm_HandSolder, F.Cu at (267.4, 47.3)
- added R24: 22K, Resistor_SMD:R_0603_1608Metric_Pad0.98x0.95mm_HandSolder, F.Cu at (271.7, 24.7)
- added R25: 22K, Resistor_SMD:R_0603_1608Metric_Pad0.98x0.95mm_HandSolder, F.Cu at (271.7, 27.2)
- added R26: 1.5K, Resistor_SMD:R_0603_1608Metric_Pad0.98x0.95mm_HandSolder, F.Cu at (271.7, 29.7)
- added R27: 1.5K, Resistor_SMD:R_0603_1608Metric_Pad0.98x0.95mm_HandSolder, F.Cu at (271.7, 32.2)
- added R28: 1.5K, Resistor_SMD:R_0603_1608Metric_Pad0.98x0.95mm_HandSolder, F.Cu at (271.7, 34.7)
- added R29: 22K, Resistor_SMD:R_0603_1608Metric_Pad0.98x0.95mm_HandSolder, F.Cu at (271.7, 37.2)
- added R30: 5.1K, Resistor_SMD:R_0603_1608Metric_Pad0.98x0.95mm_HandSolder, F.Cu at (271.7, 39.7)
- added R31: 1, Resistor_SMD:R_0603_1608Metric_Pad0.98x0.95mm_HandSolder, F.Cu at (271.7, 42.2)
- added R32: 1, Resistor_SMD:R_0603_1608Metric_Pad0.98x0.95mm_HandSolder, F.Cu at (271.7, 44.8)
- added R33: 1.5K, Resistor_SMD:R_0603_1608Metric_Pad0.98x0.95mm_HandSolder, F.Cu at (271.7, 47.3)
- added R34: 22K, Resistor_SMD:R_0603_1608Metric_Pad0.98x0.95mm_HandSolder, F.Cu at (276.1, 24.7)
- added R35: 1.5K, Resistor_SMD:R_0603_1608Metric_Pad0.98x0.95mm_HandSolder, F.Cu at (276.1, 27.2)
- added R36: 1.5K, Resistor_SMD:R_0603_1608Metric_Pad0.98x0.95mm_HandSolder, F.Cu at (276.1, 29.7)
- added R38: 1.5K, Resistor_SMD:R_0603_1608Metric_Pad0.98x0.95mm_HandSolder, F.Cu at (276.1, 32.2)
- added R39: 22K, Resistor_SMD:R_0603_1608Metric_Pad0.98x0.95mm_HandSolder, F.Cu at (276.1, 34.7)
- added R40: 5.1K, Resistor_SMD:R_0603_1608Metric_Pad0.98x0.95mm_HandSolder, F.Cu at (276.1, 37.2)
- added R41: 1, Resistor_SMD:R_0603_1608Metric_Pad0.98x0.95mm_HandSolder, F.Cu at (276.1, 39.7)
- added R42: 1, Resistor_SMD:R_0603_1608Metric_Pad0.98x0.95mm_HandSolder, F.Cu at (276.1, 42.2)
- added R43: 1.5K, Resistor_SMD:R_0603_1608Metric_Pad0.98x0.95mm_HandSolder, F.Cu at (276.1, 44.8)
- added R5: 1M, Resistor_SMD:R_0603_1608Metric_Pad0.98x0.95mm_HandSolder, F.Cu at (108.8, 84.5)
- added R6: 84.5K, Resistor_SMD:R_0603_1608Metric_Pad0.98x0.95mm_HandSolder, F.Cu at (107.1, 84.5)
- added R7: 22K, Resistor_SMD:R_0603_1608Metric_Pad0.98x0.95mm_HandSolder, F.Cu at (263.0, 37.2)
- added R8: 22K, Resistor_SMD:R_0603_1608Metric_Pad0.98x0.95mm_HandSolder, F.Cu at (263.0, 39.7)
- added R9: 22K, Resistor_SMD:R_0603_1608Metric_Pad0.98x0.95mm_HandSolder, F.Cu at (263.0, 42.2)
- added TP1: +5V, TestPoint:TestPoint_Pad_1.0x1.0mm, F.Cu at (260.3, 61.8)
- added TP2: +16V, TestPoint:TestPoint_Pad_1.0x1.0mm, F.Cu at (260.3, 64.8)
- added TP3: +3.7V, TestPoint:TestPoint_Pad_1.0x1.0mm, F.Cu at (260.3, 67.9)
- added TP4: +15VA, TestPoint:TestPoint_Pad_1.0x1.0mm, F.Cu at (260.3, 70.9)
- added TP5: VREF, TestPoint:TestPoint_Pad_1.0x1.0mm, F.Cu at (260.3, 74.0)
- added U10: NE5532, Package_SO:SOIC-8_5.3x5.3mm_P1.27mm, F.Cu at (238.3, 61.7)
- added U11: NE5532, Package_SO:SOIC-8_5.3x5.3mm_P1.27mm, F.Cu at (238.3, 68.7)
- added U5: NE5532, Package_SO:SOIC-8_5.3x5.3mm_P1.27mm, F.Cu at (238.3, 26.9)
- added U6: NE5532, Package_SO:SOIC-8_5.3x5.3mm_P1.27mm, F.Cu at (238.3, 33.9)
- added U7: NE5532, Package_SO:SOIC-8_5.3x5.3mm_P1.27mm, F.Cu at (238.3, 40.9)
- added U8: NE5532, Package_SO:SOIC-8_5.3x5.3mm_P1.27mm, F.Cu at (238.3, 47.8)
- added U9: NE5532, Package_SO:SOIC-8_5.3x5.3mm_P1.27mm, F.Cu at (238.3, 54.8)
- added Y3: 12 MHz Crystal, Crystal:Crystal_SMD_3225-4Pin_3.2x2.5mm, F.Cu at (256.0, 77.3)
- U1: value PCM2906 -> PCM2900C
- moved R3 200.4 mm to (250.2, 54.2)
- moved U3 189.4 mm to (264.4, 67.3)
- moved U1 176.3 mm to (276.6, 66.1)
- moved D5 156.2 mm to (237.2, 78.9)
- moved J2 127.6 mm to (265.6, 54.4)
- moved D4 67.7 mm to (113.4, 88.1), turned to -90 degrees
- moved U4 64.5 mm to (141.2, 49.5)
- moved U2 61.1 mm to (109.3, 88.0), turned to 180 degrees
Connections:
- J2 pad 1: unconnected-(J2-Pad1) -> GND
- J2 pad 2: unconnected-(J2-Pad2) -> Net-(D6-A2)
- J2 pad 3: unconnected-(J2-Pad3) -> Net-(D7-A2)
- U1 pad 24: Net-(U1-DIN) -> GND
- U1 pad 28: Net-(U1-~{SSPND}) -> unconnected-(U1-~{SSPND}-Pad28)
- U1 pad 5: Net-(U1-HID0) -> unconnected-(U1-HID0-Pad5)
Routing:
- net +16VA: track 0.00 -> 9.01 mm
- net +15V: track 0.00 -> 4.39 mm
- net Net-(U4-ADJ): track 0.00 -> 4.19 mm
Other:
- copper layers 2 -> 4
