File: USB_DAC-AMP_V2_different_layout/USB_DAC-AMP_V2_different_layout.kicad_pcb (KiCad board)
At the start: 4 copper layers, 121 parts, among them J1 USB_C_Receptacle, J2 SJ-3524-SMT, U1 PCM2900C, U10 NE5532, U11 NE5532, U2 TPS61040DBV, U3 SPX3819M5-L, U4 SPX3819M5-L, U5 NE5532, U6 NE5532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

Commit message: created V4 to change board dimensions, update schematic
changed out caps to be electrolytic
board dimensions are now whole numbers
Parts:
- added C47: 100n, Capacitor_SMD:C_0603_1608Metric_Pad1.08x0.95mm_HandSolder, F.Cu at (145.9, 107.4)
- C27: value 1000u -> 100u
- R17: value 2.2 -> 1
- moved R31 201.4 mm to (101.4, 149.8)
- moved R32 201.4 mm to (101.4, 152.3)
- moved R33 201.4 mm to (101.4, 154.8)
- moved R27 195.4 mm to (101.1, 127.5), turned to -90 degrees
- moved R26 188.7 mm to (100.5, 108.8), turned to -90 degrees
- moved R28 188.6 mm to (104.4, 121.8), turned to 180 degrees
- moved FB4 186.4 mm to (101.4, 147.2)
- moved R29 184.9 mm to (111.4, 129.3)
- moved D6 184.6 mm to (105.8, 155.1)
- moved C34 182.7 mm to (101.4, 142.2)
- moved C36 182.7 mm to (101.4, 144.7)
- moved R30 181.0 mm to (112.6, 126.0), turned to -90 degrees
- moved R34 177.5 mm to (143.3, 142.4)
- moved R35 177.5 mm to (143.3, 145.0)
- moved R23 171.2 mm to (104.5, 100.0)
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Routing:
- net +5V: track 18.9 -> 43.1 mm, vias 0 -> 2
- net +15V: track 24.9 -> 4.39 mm, vias 2 -> 0
- net VREF: track 18.9 -> 0.00 mm
- net +15VA: track 32.5 -> 17.5 mm
- net VDDI: track 13.9 -> 28.7 mm, vias 0 -> 2
- net Net-(U5A--): track 0.00 -> 13.8 mm
- net Net-(U9B--): track 0.00 -> 11.6 mm
- net Net-(U1-VINL): track 0.00 -> 9.32 mm
- net Net-(U5B--): track 0.00 -> 8.21 mm
- net +16V: track 20.8 -> 13.4 mm, vias 2 -> 0
- net Net-(U1-VINR): track 0.00 -> 6.53 mm
- net Net-(U9A-+): track 0.00 -> 5.75 mm
- net Net-(U5A-+): track 0.00 -> 5.69 mm
- net Net-(U9A--): track 0.00 -> 5.61 mm
- net Net-(U7A-+): track 0.00 -> 4.10 mm
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