File: USB_DAC-AMP_V2_different_layout/USB_DAC-AMP_V2_different_layout.kicad_sch (KiCad schematic)
At the start: 121 parts, among them J1 USB_C_Receptacle, J2 SJ-3524-SMT, U1 PCM2900C, U10 NE5532, U11 NE5532, U2 TPS61040DBV, U3 SPX3819M5-L, U4 SPX3819M5-L, U5 NE5532, U6 NE5532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

Commit message: created V4 to change board dimensions, update schematic
changed out caps to be electrolytic
board dimensions are now whole numbers
Parts:
- added C47: 100n, Capacitor_SMD:C_0603_1608Metric_Pad1.08x0.95mm_HandSolder, symbol Device:C
- added H1, H2, H3, H4: MountingHole, symbol Mechanical:MountingHole
- C27: value 1000u -> 100u
- R17: value 2.2 -> 1
Connections:
- net GND: now also C47.1
- net VREF: now also C47.2
Other:
- moved on the sheet: C27
