File: USB_DAC-AMP_V3_iPhone_dimensions/USB_DAC-AMP_V3_iPhone_dimensions.kicad_sch (KiCad schematic)
At the start: 121 parts, among them J1 USB_C_Receptacle, J2 SJ-3524-SMT, U1 PCM2900C, U10 NE5532, U11 NE5532, U2 TPS61040DBV, U3 SPX3819M5-L, U4 SPX3819M5-L, U5 NE5532, U6 NE5532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

Commit message: created V4 to change board dimensions, update schematic
changed out caps to be electrolytic
board dimensions are now whole numbers
Parts:
- added C47: 100n, Capacitor_SMD:C_0603_1608Metric_Pad1.08x0.95mm_HandSolder, symbol Device:C
- added H1, H2, H3, H4: MountingHole, MountingHole:MountingHole_3.5mm, symbol Mechanical:MountingHole
- C1, C10, C11, C12, C13, C19, C9: LCSC (none) -> C1035
- C14, C15, C35, C45: LCSC (none) -> C696799
- C16, C17, C18, C20, C21, C22, C7, C8: LCSC (none) -> C1592
- C2, C23, C24, C3, C33, C36, C4, C43, C46, C5, C6: LCSC (none) -> C1658
- C25, C30, C31, C40, C41: LCSC (none) -> C132558
- C26, C28, C32, C34, C38, C42, C44: LCSC (none) -> C1590
- C27: value 1000u -> 100u; LCSC (none) -> C132558
- C29, C39: LCSC (none) -> C1028
- C37: LCSC (none) -> C1002
- R17: value 2.2 -> 1
- R20, R21: value 1.5k -> 5.1K
- R3: footprint PTN092-H20115K1A:TRIM_PTN092-H20115K1A -> Imported_footprints:TRIM_PTN092-H20115K1A
Connections:
- net +16V: now also FB2.2; no longer FB2.1
- net +16VA: now also FB2.1; no longer FB2.2
- net GND: now also C47.1
- net VBL: no longer R36.2, R39.2
- net VBR: now also R36.2, R39.2
- net VREF: now also C47.2
- net at C41.2: now also R3.2_1; no longer R3.2_2
- net at C43.2, R40.1, U10.7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: now also R3.3_1; no longer R3.3_2
- net at C35.1, R32.1: now also R31.2; no longer R31.1
- net at U8.1, U8.2 (-): now also R26.2; no longer R35.1
- net at C39.2, U8.5 (+): now also R26.1; no longer R35.2
- net at C29.2, U5.5 (+): now also R35.2; no longer R26.2
- net at C33.2, R30.1, U7.3 (+)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: now also R3.3_2, U7.5 (+); no longer R3.3_1, U7.6 (-)
- net at U7.1, U7.2 (-): now also R31.1; no longer R31.2
- net at C31.2: now also R3.2_2; no longer R3.2_1
- net at R32.2, U7.7: now also U7.6 (-); no longer U7.5 (+)
- net at C40.2: now also R3.1_1; no longer R3.1_2
- net at U5.1, U5.2 (-): now also R35.1; no longer R26.1
- net at C30.2: now also R3.1_2; no longer R3.1_1
Other:
- moved on the sheet: C27, C31, FB2, R26, R31, R35
