File: USB_DAC-AMP_V4_credit_card/USB_DAC-AMP_V4_credit_card.kicad_pcb (KiCad board)
At the start: 4 copper layers, 70.7 x 88.2 mm, 126 parts, among them J1 USB_C_Receptacle, J2 SJ-3524-SMT, U1 PCM2900C, U10 NE5532, U11 NE5532, U2 TPS61040DBV, U3 SPX3819M5-L, U4 SPX3819M5-L, U5 NE5532, U6 NE5532, U7 NE5532, U8 NE5532, U9 NE5532, Y3 12 MHz Crystal

Commit message: updated V4
Parts:
- removed C46: 30p, Capacitor_SMD:C_0603_1608Metric_Pad1.08x0.95mm_HandSolder
- removed C47: 100n, Capacitor_SMD:C_0603_1608Metric_Pad1.08x0.95mm_HandSolder
- removed R40: 5.1K, Resistor_SMD:R_0603_1608Metric_Pad0.98x0.95mm_HandSolder
- removed R41, R42: 1, Resistor_SMD:R_0603_1608Metric_Pad0.98x0.95mm_HandSolder
- removed R43: 1.5K, Resistor_SMD:R_0603_1608Metric_Pad0.98x0.95mm_HandSolder
- removed Y3: 12 MHz Crystal, Crystal:Crystal_SMD_3225-4Pin_3.2x2.5mm
- added R18: 22, Resistor_SMD:R_0603_1608Metric, F.Cu at (92.8, 41.6)
- added R19: 1, Resistor_SMD:R_0603_1608Metric, F.Cu at (80.0, 88.6)
- added R37: 1.5K, Resistor_SMD:R_0603_1608Metric, F.Cu at (213.7, 53.4)
- added R4: 1.5K, Resistor_SMD:R_0603_1608Metric, F.Cu at (138.0, 104.6)
- added Y1: 12 MHz Crystal, Crystal:Crystal_SMD_3225-4Pin_3.2x2.5mm, F.Cu at (104.4, 48.8)
- C1, C11, C19: value 10u -> 1u; footprint Capacitor_SMD:C_0603_1608Metric_Pad1.08x0.95mm_HandSolder -> Capacitor_SMD:C_0603_1608Metric
- C10, C12, C13, C9: value 10u -> 30p; footprint Capacitor_SMD:C_0603_1608Metric_Pad1.08x0.95mm_HandSolder -> Capacitor_SMD:C_0603_1608Metric
- C14: value 1000u -> 1u; footprint Capacitor_Tantalum_SMD:CP_EIA-7343-43_Kemet-X_HandSolder -> Capacitor_SMD:C_0603_1608Metric
- C15: value 1000u -> 30p; footprint Capacitor_Tantalum_SMD:CP_EIA-7343-43_Kemet-X_HandSolder -> Capacitor_SMD:C_0603_1608Metric
- C16: value 1u -> 30p; footprint Capacitor_SMD:C_0603_1608Metric_Pad1.08x0.95mm_HandSolder -> Capacitor_SMD:C_0603_1608Metric
- C17, C18, C22, C8: value 1u -> 10u; footprint Capacitor_SMD:C_0603_1608Metric_Pad1.08x0.95mm_HandSolder -> Capacitor_SMD:C_0603_1608Metric
- C2, C23: value 30p -> 1u; footprint Capacitor_SMD:C_0603_1608Metric_Pad1.08x0.95mm_HandSolder -> Capacitor_SMD:C_0603_1608Metric
- C20, C21, C34, C4, C43: footprint Capacitor_SMD:C_0603_1608Metric_Pad1.08x0.95mm_HandSolder -> Capacitor_SMD:C_0603_1608Metric
- C24, C33, C36: value 30p -> 100n; footprint Capacitor_SMD:C_0603_1608Metric_Pad1.08x0.95mm_HandSolder -> Capacitor_SMD:C_0603_1608Metric
- C25: value 100u -> 100n; footprint Capacitor_Tantalum_SMD:CP_EIA-7343-43_Kemet-X_HandSolder -> Capacitor_SMD:C_0603_1608Metric
- C26, C38: value 100n -> 1000u; footprint Capacitor_SMD:C_0603_1608Metric_Pad1.08x0.95mm_HandSolder -> Capacitor_SMD:CP_Elec_10x10.5
- C27, C41: footprint Capacitor_Tantalum_SMD:CP_EIA-7343-43_Kemet-X_HandSolder -> Capacitor_SMD:CP_Elec_6.3x7.7
- C28: value 100n -> 30p; footprint Capacitor_SMD:C_0603_1608Metric_Pad1.08x0.95mm_HandSolder -> Capacitor_SMD:C_0603_1608Metric
- C29, C39: value 2.2n -> 100u; footprint Capacitor_SMD:C_0603_1608Metric_Pad1.08x0.95mm_HandSolder -> Capacitor_SMD:CP_Elec_6.3x7.7
- C3, C5, C6: value 30p -> 10u; footprint Capacitor_SMD:C_0603_1608Metric_Pad1.08x0.95mm_HandSolder -> Capacitor_SMD:C_0603_1608Metric
- C30: value 100u -> 2.2n; footprint Capacitor_Tantalum_SMD:CP_EIA-7343-43_Kemet-X_HandSolder -> Capacitor_SMD:C_0603_1608Metric
- C31, C40: value 100u -> 30p; footprint Capacitor_Tantalum_SMD:CP_EIA-7343-43_Kemet-X_HandSolder -> Capacitor_SMD:C_0603_1608Metric
- C32, C44: value 100n -> 100u; footprint Capacitor_SMD:C_0603_1608Metric_Pad1.08x0.95mm_HandSolder -> Capacitor_SMD:CP_Elec_6.3x7.7
- C35: value 1000u -> 100u; footprint Capacitor_Tantalum_SMD:CP_EIA-7343-43_Kemet-X_HandSolder -> Capacitor_SMD:CP_Elec_6.3x7.7
- C37: value 100u -> 100n; footprint Capacitor_Tantalum_SMD:CP_EIA-7343-15_Kemet-W -> Capacitor_SMD:C_0603_1608Metric
- C42: value 100n -> 2.2n; footprint Capacitor_SMD:C_0603_1608Metric_Pad1.08x0.95mm_HandSolder -> Capacitor_SMD:C_0603_1608Metric
- C45: value 1000u -> 100n; footprint Capacitor_Tantalum_SMD:CP_EIA-7343-43_Kemet-X_HandSolder -> Capacitor_SMD:C_0603_1608Metric
- C7: value 1u -> 100u; footprint Capacitor_SMD:C_0603_1608Metric_Pad1.08x0.95mm_HandSolder -> Capacitor_SMD:CP_Elec_6.3x7.7
- D1: value D_TVS -> SS14; footprint Diode_SMD:D_0603_1608Metric_Pad1.05x0.95mm_HandSolder -> Diode_SMD:D_SMA
- D2: value 0603ESDA-18N -> LED; footprint Diode_SMD:D_0603_1608Metric_Pad1.05x0.95mm_HandSolder -> LED_SMD:LED_0603_1608Metric
- D3: value LED -> D_TVS; footprint LED_SMD:LED_0603_1608Metric_Pad1.05x0.95mm_HandSolder -> Diode_SMD:D_0603_1608Metric
- D4: value SS14 -> D_TVS; footprint Diode_SMD:D_SMA -> Diode_SMD:D_0603_1608Metric
- D6, D7: footprint Diode_SMD:D_0603_1608Metric_Pad1.05x0.95mm_HandSolder -> Diode_SMD:D_0603_1608Metric
- F1: footprint Fuse:Fuse_0603_1608Metric_Pad1.05x0.95mm_HandSolder -> Fuse:Fuse_0603_1608Metric
- FB1, FB2, FB3, FB4, FB5, R16, R26, R29, R31, R33, R36, R39, R8: footprint Resistor_SMD:R_0603_1608Metric_Pad0.98x0.95mm_HandSolder -> Resistor_SMD:R_0603_1608Metric
- L1: footprint Inductor_SMD:L_0805_2012Metric_Pad1.05x1.20mm_HandSolder -> Inductor_SMD:L_0805_2012Metric
- R1: value 5.1K -> 20; footprint Resistor_SMD:R_0603_1608Metric_Pad0.98x0.95mm_HandSolder -> Resistor_SMD:R_0603_1608Metric
- R10: value 240K -> 1M; footprint Resistor_SMD:R_0603_1608Metric_Pad0.98x0.95mm_HandSolder -> Resistor_SMD:R_0603_1608Metric
- R11, R24: value 22K -> 5.1K; footprint Resistor_SMD:R_0603_1608Metric_Pad0.98x0.95mm_HandSolder -> Resistor_SMD:R_0603_1608Metric
- R12: value 20 -> 5.1K; footprint Resistor_SMD:R_0603_1608Metric_Pad0.98x0.95mm_HandSolder -> Resistor_SMD:R_0603_1608Metric
- R13, R28: value 1.5K -> 22K; footprint Resistor_SMD:R_0603_1608Metric_Pad0.98x0.95mm_HandSolder -> Resistor_SMD:R_0603_1608Metric
- R14, R15: value 22 -> 22K; footprint Resistor_SMD:R_0603_1608Metric_Pad0.98x0.95mm_HandSolder -> Resistor_SMD:R_0603_1608Metric
- R17: value 1 -> 22; footprint Resistor_SMD:R_0603_1608Metric_Pad0.98x0.95mm_HandSolder -> Resistor_SMD:R_0603_1608Metric
- R2: value 5.1K -> 1M; footprint Resistor_SMD:R_0603_1608Metric_Pad0.98x0.95mm_HandSolder -> Resistor_SMD:R_0603_1608Metric
- R20: value 1.5k -> 22K; footprint Resistor_SMD:R_0603_1608Metric_Pad0.98x0.95mm_HandSolder -> Resistor_SMD:R_0603_1608Metric
- R21: value 1.5k -> PTN092-H20115K1A; footprint Resistor_SMD:R_0603_1608Metric_Pad0.98x0.95mm_HandSolder -> Imported_footprints:TRIM_PTN092-H20115K1A
- R22: value 1M -> 1.5K; footprint Resistor_SMD:R_0603_1608Metric_Pad0.98x0.95mm_HandSolder -> Resistor_SMD:R_0603_1608Metric
- R23, R25, R34: value 22K -> 1.5K; footprint Resistor_SMD:R_0603_1608Metric_Pad0.98x0.95mm_HandSolder -> Resistor_SMD:R_0603_1608Metric
- R27, R38: value 1.5K -> 1; footprint Resistor_SMD:R_0603_1608Metric_Pad0.98x0.95mm_HandSolder -> Resistor_SMD:R_0603_1608Metric
- R3: value PTN092-H20115K1A -> 240K; footprint Imported_footprints:TRIM_PTN092-H20115K1A -> Resistor_SMD:R_0603_1608Metric
- R30: value 5.1K -> 22K; footprint Resistor_SMD:R_0603_1608Metric_Pad0.98x0.95mm_HandSolder -> Resistor_SMD:R_0603_1608Metric
- R32: value 1 -> 22K; footprint Resistor_SMD:R_0603_1608Metric_Pad0.98x0.95mm_HandSolder -> Resistor_SMD:R_0603_1608Metric
- R35: value 1.5K -> 5.1K; footprint Resistor_SMD:R_0603_1608Metric_Pad0.98x0.95mm_HandSolder -> Resistor_SMD:R_0603_1608Metric
- R5: value 1M -> 5.1K; footprint Resistor_SMD:R_0603_1608Metric_Pad0.98x0.95mm_HandSolder -> Resistor_SMD:R_0603_1608Metric
- R6: value 84.5K -> 5.1K; footprint Resistor_SMD:R_0603_1608Metric_Pad0.98x0.95mm_HandSolder -> Resistor_SMD:R_0603_1608Metric
- R7: value 22K -> 84.5K; footprint Resistor_SMD:R_0603_1608Metric_Pad0.98x0.95mm_HandSolder -> Resistor_SMD:R_0603_1608Metric
- R9: value 22K -> 1; footprint Resistor_SMD:R_0603_1608Metric_Pad0.98x0.95mm_HandSolder -> Resistor_SMD:R_0603_1608Metric
- TP3: value +3.7V -> +15VA
- TP4: value +15VA -> +3.7V
- TP5: value VREF -> U1_VCCI
- TP6: value U1_VCCI -> VBL
- TP7: value VBL -> VREF
- U1: value PCM2900C -> TPS61040DBV; footprint Package_SO:SSOP-28_5.3x10.2mm_P0.65mm -> Package_TO_SOT_SMD:SOT-23-5
- U2: value TPS61040DBV -> SPX3819M5-L
- U4: value SPX3819M5-L -> PCM2900C; footprint Package_TO_SOT_SMD:SOT-23-5 -> Package_SO:SSOP-28_5.3x10.2mm_P0.65mm
- moved C27 142.3 mm to (73.2, 78.2), turned to 180 degrees
- moved C30 135.9 mm to (83.8, 64.4)
- moved C25 132.6 mm to (83.0, 72.0), turned to 180 degrees
- moved C35 130.8 mm to (95.0, 60.4), turned to 180 degrees
- moved R13 130.5 mm to (69.2, 36.8), turned to 90 degrees
- moved R32 127.5 mm to (213.7, 40.8), turned to 0 degrees
- moved C41 125.1 mm to (103.2, 68.2), turned to 180 degrees
- moved C31 124.9 mm to (93.0, 78.4), turned to 90 degrees
- moved C14 120.3 mm to (99.0, 44.4)
- moved C15 118.8 mm to (101.8, 46.6), turned to -90 degrees
- moved D3 118.6 mm to (92.6, 35.2)
- moved R31 116.9 mm to (209.4, 68.4), turned to 0 degrees
- moved H3 116.8 mm to (63.8, 111.2)
- moved R35 113.0 mm to (213.7, 48.3), turned to 0 degrees
- moved H2 111.0 mm to (126.2, 28.8)
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Connections:
- C1 pad 1: +5V -> Net-(C1-Pad1)
- C10 pad 1: Net-(U3-EN) -> Net-(J1-CC2)
- C11 pad 1: +3.7V -> Net-(U4-VBUS)
- C12 pad 1: +16VA -> /D+
- C13 pad 1: +15V -> /D-
- C14 pad 1: +15VA -> VDDI
- C15 pad 1: +15VA -> Net-(U4-XTI)
- C16 pad 1: VDDI -> Net-(U4-XTO)
- C17 pad 1: Net-(U1-VBUS) -> Net-(U3-EN)
- C18 pad 1: Net-(D5-K) -> +3.7V
- C19 pad 1: Net-(U1-VCOM) -> Net-(U4-VCCXI)
- C2 pad 1: Net-(J1-CC2) -> +5V
- C20 pad 1: Net-(U1-VCCP1I) -> Net-(U4-VCCP2I)
- C21 pad 1: Net-(U1-VCCP2I) -> Net-(U4-VCCP1I)
- C22 pad 1: Net-(U1-VCCXI) -> Net-(U4-VCOM)
- C23 pad 1: Net-(U1-XTO) -> Net-(D5-K)
- C24 pad 1: Net-(U1-XTI) -> +15VA
- C25 pad 1: /VOUTL -> +15VA
- C25 pad 2: Net-(U5A-+) -> GND
- C26 pad 1: +15VA -> Net-(C26-Pad1)
- C26 pad 2: GND -> Net-(C26-Pad2)
- C27 pad 1: GND -> Net-(U6B--)
- C27 pad 2: VREF -> Net-(C27-Pad2)
- C28 pad 1: +15VA -> GND
- C28 pad 2: GND -> Net-(D6-A2)
- C29 pad 1: GND -> Net-(U6A-+)
- C29 pad 2: Net-(U5B-+) -> /VOUTL
- C3 pad 1: Net-(J1-CC1) -> +5V
- C30 pad 1: Net-(U5B--) -> GND
- C30 pad 2: Net-(C30-Pad2) -> Net-(U6B-+)
- C31 pad 1: Net-(U9A-+) -> Net-(U7B--)
- C31 pad 2: Net-(C31-Pad2) -> Net-(U5A-+)
- C32 pad 1: +15VA -> Net-(U7A-+)
- C32 pad 2: GND -> Net-(C32-Pad2)
- C33 pad 1: Net-(U9B--) -> +15VA
- C33 pad 2: Net-(U7A-+) -> GND
- C35 pad 1: Net-(C35-Pad1) -> VREF
- C35 pad 2: Net-(C35-Pad2) -> GND
- C36 pad 1: GND -> +15VA
- C36 pad 2: Net-(D6-A2) -> GND
- C37 pad 1: /VOUTR -> +15VA
- C37 pad 2: Net-(U8A-+) -> GND
- C38 pad 1: +15VA -> Net-(C38-Pad1)
- C38 pad 2: GND -> Net-(C38-Pad2)
- C39 pad 1: GND -> Net-(U10B--)
- C39 pad 2: Net-(U8B-+) -> Net-(C39-Pad2)
- C4 pad 1: /D+ -> +16V
- C4 pad 2: GND -> Net-(U1-FB)
- C40 pad 1: Net-(U8B--) -> GND
- C40 pad 2: Net-(C40-Pad2) -> Net-(D7-A2)
- C41 pad 2: Net-(C41-Pad2) -> /VOUTR
- C42 pad 1: +15VA -> GND
- C42 pad 2: GND -> Net-(U10B-+)
- C43 pad 1: Net-(U10B--) -> Net-(U11B--)
- C43 pad 2: Net-(U11A-+) -> Net-(U9A-+)
- C44 pad 1: +15VA -> Net-(U11A-+)
- C44 pad 2: GND -> Net-(C44-Pad2)
- C45 pad 1: Net-(C45-Pad1) -> +15VA
- C45 pad 2: Net-(C45-Pad2) -> GND
- C5 pad 1: /D- -> +16V
- C6 pad 1: +16V -> +16VA
- C6 pad 2: Net-(U2-FB) -> GND
- C7 pad 1: Net-(C7-Pad1) -> +15VA
- C8 pad 1: +5V -> +15V
- C9 pad 1: +16V -> Net-(J1-CC1)
- D1 pad 1: GND -> +16V
- D1 pad 2: /D+ -> Net-(D1-A)
- D2 pad 1: GND -> Net-(D2-K)
- D2 pad 2: /D- -> +15VA
- D3 pad 1: Net-(D3-K) -> GND
- D3 pad 2: +15VA -> /D+
- D4 pad 1: +16V -> GND
- D4 pad 2: Net-(D4-A) -> /D-
- F1 pad 2: Net-(C7-Pad1) -> Net-(C1-Pad1)
- FB1 pad 1: Net-(C7-Pad1) -> Net-(C1-Pad1)
- FB4 pad 1: Net-(C35-Pad2) -> Net-(C26-Pad2)
- FB5 pad 1: Net-(C45-Pad2) -> Net-(C38-Pad2)
- L1 pad 2: Net-(D4-A) -> Net-(D1-A)
- R1 pad 1: Net-(J1-CC1) -> +15V
- R1 pad 2: GND -> +15VA
- R10 pad 1: +15V -> Net-(U4-XTI)
- R10 pad 2: Net-(U4-ADJ) -> Net-(U4-XTO)
- R11 pad 1: Net-(U4-ADJ) -> GND
- R11 pad 2: GND -> Net-(U4-VINL)
- R12 pad 1: +15V -> GND
- R12 pad 2: +15VA -> Net-(U4-VINR)
- R13 pad 1: Net-(D3-K) -> +3.7V
- R13 pad 2: GND -> Net-(U3-ADJ)
- R14 pad 1: /D+ -> Net-(U3-ADJ)
- R14 pad 2: Net-(U1-D+) -> GND
- R15 pad 1: /D- -> Net-(U3-ADJ)
- R15 pad 2: Net-(U1-D-) -> GND
- R17 pad 1: +5V -> /D+
- R17 pad 2: Net-(U1-VBUS) -> Net-(U4-D+)
- R2 pad 1: Net-(J1-CC2) -> +16V
- R2 pad 2: GND -> Net-(U1-FB)
- R20 pad 1: GND -> VBL
- R20 pad 2: Net-(U1-VINL) -> Net-(U6A-+)
- R22 pad 1: Net-(U1-XTI) -> Net-(U6A--)
- R22 pad 2: Net-(U1-XTO) -> Net-(U6B-+)
- R23 pad 1: VBL -> Net-(C26-Pad2)
- R23 pad 2: Net-(U5A-+) -> GND
- R24 pad 1: +15VA -> Net-(U5A-+)
- R24 pad 2: VREF -> Net-(U7B--)
- R25 pad 1: VREF -> Net-(U7A-+)
- R25 pad 2: GND -> VBL
- R26 pad 1: Net-(U8B-+) -> Net-(U7B--)
- R26 pad 2: Net-(U8A--) -> Net-(U7A--)
- R27 pad 1: Net-(U9A-+) -> Net-(C26-Pad1)
- R27 pad 2: VBL -> Net-(U5B--)
- R28 pad 1: Net-(U9B--) -> Net-(U7B-+)
- R28 pad 2: Net-(U9A--) -> VBL
- R29 pad 1: Net-(U9B-+) -> +15VA
- R29 pad 2: VBL -> VREF
- R30 pad 1: Net-(U7A-+) -> VREF
- R30 pad 2: Net-(U9B--) -> GND
- R31 pad 1: Net-(U7A--) -> Net-(C38-Pad1)
- R31 pad 2: Net-(C35-Pad1) -> Net-(U9A--)
- R32 pad 1: Net-(C35-Pad1) -> VBR
- R32 pad 2: Net-(U7B--) -> Net-(U10A-+)
- R33 pad 1: Net-(C35-Pad2) -> Net-(U10B-+)
- R33 pad 2: GND -> Net-(U10A--)
- R34 pad 1: VBR -> Net-(C38-Pad2)
- R34 pad 2: Net-(U8A-+) -> GND
- R35 pad 1: Net-(U5A--) -> Net-(U9A-+)
- R35 pad 2: Net-(U5B-+) -> Net-(U11B--)
- R36 pad 1: Net-(U10A-+) -> Net-(U11A-+)
- R38 pad 1: Net-(U10B--) -> Net-(C38-Pad1)
- R38 pad 2: Net-(U10A--) -> Net-(U9B--)
- R39 pad 1: Net-(U10B-+) -> Net-(U11B-+)
- R5 pad 1: +16V -> Net-(J1-CC1)
- R5 pad 2: Net-(U2-FB) -> GND
- R6 pad 1: Net-(U2-FB) -> Net-(J1-CC2)
- R7 pad 1: +3.7V -> Net-(U1-FB)
- R7 pad 2: Net-(U3-ADJ) -> GND
- R8 pad 1: Net-(U3-ADJ) -> Net-(U2-ADJ)
- R9 pad 1: Net-(U3-ADJ) -> +5V
- R9 pad 2: GND -> Net-(U4-VBUS)
- TP3 pad 1: +3.7V -> +15VA
- TP4 pad 1: +15VA -> +3.7V
- TP5 pad 1: VREF -> Net-(D5-K)
- TP6 pad 1: Net-(D5-K) -> VBL
- TP7 pad 1: VBL -> VREF
- U1 pad 1: Net-(U1-D+) -> Net-(D1-A)
- U1 pad 2: Net-(U1-D-) -> GND
- U1 pad 3: Net-(U1-VBUS) -> Net-(U1-FB)
- U1 pad 4: GND -> +5V
- U1 pad 5: unconnected-(U1-HID0-Pad5) -> +5V
- U10 pad 7: Net-(U11A-+) -> Net-(U10B--)
- U11 pad 5: Net-(U11A-+) -> Net-(U11B-+)
- U11 pad 7: Net-(U11B--) -> Net-(U9A-+)
- U2 pad 1: Net-(D4-A) -> +16VA
- U2 pad 3: Net-(U2-FB) -> +16VA
- U2 pad 4: +5V -> Net-(U2-ADJ)
- U2 pad 5: +5V -> +15V
- U4 pad 1: +16VA -> Net-(U4-D+)
- U4 pad 2: GND -> Net-(U4-D-)
- U4 pad 3: +16VA -> Net-(U4-VBUS)
- U4 pad 4: Net-(U4-ADJ) -> GND
- U4 pad 5: +15V -> unconnected-(U4-HID0-Pad5)
- U5 pad 5: Net-(U5B-+) -> Net-(U5A-+)
- U6 pad 1: VBL -> Net-(U6A--)
- U6 pad 2: VBL -> Net-(U6A--)
- U6 pad 3: VREF -> Net-(U6A-+)
- U6 pad 5: VREF -> Net-(U6B-+)
- U6 pad 6: VBR -> Net-(U6B--)
- U6 pad 7: VBR -> Net-(U6B--)
- U7 pad 5: Net-(U7A-+) -> Net-(U7B-+)
- U7 pad 7: Net-(U7B--) -> Net-(U5A-+)
- U8 pad 1: Net-(U8A--) -> VBL
- U8 pad 2: Net-(U8A--) -> VBL
- U8 pad 3: Net-(U8A-+) -> VREF
- U8 pad 5: Net-(U8B-+) -> VREF
- U8 pad 6: Net-(U8B--) -> VBR
- U8 pad 7: Net-(U8B--) -> VBR
- U9 pad 5: Net-(U9B-+) -> Net-(U9A-+)
- U9 pad 7: Net-(U7A-+) -> Net-(U9B--)
Routing:
- net +15VA: track 186.3 -> 47.5 mm
- net Net-(U11A-+): track 102.0 -> 0.00 mm, vias 3 -> 0
- net Net-(U5A-+): track 6.98 -> 73.2 mm, vias 0 -> 2
- net Net-(U7A-+): track 76.7 -> 15.9 mm, vias 1 -> 0
- net VBR: track 63.6 -> 3.37 mm, vias 3 -> 0
- net Net-(C44-Pad2): track 0.00 -> 58.0 mm, vias 0 -> 1
- net Net-(U9A-+): track 6.97 -> 63.3 mm, vias 0 -> 3
- net Net-(C41-Pad2): track 55.7 -> 0.00 mm, vias 1 -> 0
- net Net-(C39-Pad2): track 0.00 -> 49.8 mm, vias 0 -> 1
- net Net-(C40-Pad2): track 47.0 -> 0.00 mm, vias 1 -> 0
- net Net-(C32-Pad2): track 0.00 -> 44.4 mm, vias 0 -> 1
- net Net-(C27-Pad2): track 0.00 -> 36.3 mm, vias 0 -> 1
- net Net-(C31-Pad2): track 30.6 -> 0.00 mm, vias 1 -> 0
- net Net-(D7-A2): track 23.1 -> 0.00 mm
- net Net-(C30-Pad2): track 22.7 -> 0.00 mm, vias 1 -> 0
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Other:
- board size 70.7 x 88.2 mm -> 70 x 90 mm
- board text removed: "Ishaan Tamarapalli USB_DAC-AMP V1"

Commit message: Finished V4 layout
Parts:
- added TP11: buffer2_r, TestPoint:TestPoint_Pad_1.0x1.0mm, F.Cu at (120.0, 93.0)
- added TP12: buffer2_l, TestPoint:TestPoint_Pad_1.0x1.0mm, F.Cu at (78.4, 93.0)
- added TP13: in_l, TestPoint:TestPoint_Pad_1.0x1.0mm, F.Cu at (78.4, 65.8)
- added TP14: in_r, TestPoint:TestPoint_Pad_1.0x1.0mm, F.Cu at (108.2, 65.8)
- added TP15: buffer1_l, TestPoint:TestPoint_Pad_1.0x1.0mm, F.Cu at (66.6, 78.2)
- added TP16: buffer1_r, TestPoint:TestPoint_Pad_1.0x1.0mm, F.Cu at (96.8, 78.2)
- moved R34 123.6 mm to (104.8, 104.2), turned to 180 degrees
- moved FB5 107.8 mm to (104.8, 102.6), turned to 180 degrees
- moved R36 103.3 mm to (115.2, 82.0)
- moved R37 102.7 mm to (113.2, 74.4), turned to 180 degrees
- moved R31 101.4 mm to (110.0, 88.6), turned to 90 degrees
- moved C40 99.3 mm to (104.8, 99.4), turned to 180 degrees
- moved R38 98.3 mm to (121.4, 89.6), turned to 90 degrees
- moved R39 98.0 mm to (118.6, 82.0), turned to 180 degrees
- moved R35 97.1 mm to (121.4, 78.4), turned to -90 degrees
- moved R32 96.4 mm to (121.4, 68.6), turned to 90 degrees
- moved D7 96.1 mm to (104.8, 101.0), turned to 180 degrees
- moved C37 84.0 mm to (113.4, 72.0), turned to 180 degrees
- moved C36 82.8 mm to (118.6, 84.4), turned to 180 degrees
- moved C45 77.9 mm to (118.6, 74.4), turned to 180 degrees
- moved C43 74.4 mm to (123.0, 78.4), turned to 90 degrees
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Routing:
- net +15VA: track 47.5 -> 136.1 mm, vias 0 -> 2
- net VBR: track 3.37 -> 40.0 mm, vias 0 -> 3
- net Net-(C38-Pad1): track 0.00 -> 23.8 mm
- net Net-(U9A-+): track 63.3 -> 86.2 mm, vias 3 -> 4
- net Net-(D7-A2): track 0.00 -> 18.3 mm
- net Net-(U11A-+): track 0.00 -> 16.4 mm, vias 0 -> 2
- net Net-(U10B--): track 0.00 -> 16.2 mm
- net Net-(U11B--): track 0.00 -> 11.3 mm
- net Net-(U10A--): track 0.00 -> 9.35 mm
- net Net-(C26-Pad2): track 16.7 -> 7.91 mm
- net Net-(C38-Pad2): track 0.00 -> 7.91 mm
- net Net-(C26-Pad1): track 20.6 -> 28.4 mm
- net Net-(U10B-+): track 0.00 -> 6.32 mm
- net Net-(U9A--): track 0.00 -> 5.67 mm
- net Net-(U11A--): track 0.00 -> 5.21 mm
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Other:
- board text added: "Ishaan Tamarapalli USB_DAC-AMP V1"

Commit message: Submitted V1 to Kicad
Parts:
- added G***: LOGO, LOGO, B.Cu at (92.2, 75.2)
- added R40: 1.5K, Resistor_SMD:R_0603_1608Metric, F.Cu at (97.4, 43.0)
- R25, R36: value 1.5K -> 22K
- U10, U11, U5, U6, U7, U8, U9: footprint Package_SO:SOIC-8_5.3x5.3mm_P1.27mm -> Package_SO:SOIC-8_3.9x4.9mm_P1.27mm
- moved D2 24.1 mm to (107.4, 111.8), turned to 0 degrees
- moved R4 21.3 mm to (107.4, 110.0), turned to 0 degrees
- moved TP8 1.84 mm to (122.6, 70.6)
- moved C34 1.50 mm to (114.2, 54.4)
- moved TP6 1.44 mm to (114.2, 60.2)
- moved R19 1.41 mm to (81.0, 89.6)
- moved R31 1.41 mm to (111.0, 89.6)
- moved C33 1.22 mm to (87.4, 74.6)
- moved C45 1.22 mm to (117.4, 74.6)
- moved C24 1.06 mm to (87.6, 84.6)
- moved C36 1.02 mm to (117.6, 84.6)
- moved R26 1.02 mm to (84.0, 74.6)
- moved C31 1.00 mm to (92.0, 78.4)
- moved R21 1.00 mm to (67.0, 48.6)
- moved R24 1.00 mm to (90.4, 78.4)
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Connections:
- U4 pad 28: unconnected-(U4-~{SSPND}-Pad28) -> Net-(U4-~{SSPND})
Routing:
- net +15VA: track 136.1 -> 173.6 mm
- net Net-(U9A-+): track 86.2 -> 80.8 mm
- net Net-(U10A-+): track 18.3 -> 21.3 mm
- net Net-(C38-Pad1): track 23.8 -> 21.0 mm
- net Net-(C26-Pad1): track 28.4 -> 26.0 mm
- net VREF: track 35.5 -> 33.3 mm
- net GND: track 8.92 -> 11.0 mm, vias 251 -> 256
- net Net-(U5A-+): track 72.6 -> 70.6 mm
- net Net-(U7B--): track 12.2 -> 10.2 mm
- net Net-(U6A--): track 8.85 -> 10.5 mm
- net Net-(U4-~{SSPND}): track 0.00 -> 1.57 mm
- net VDDI: track 27.0 -> 28.6 mm
- net Net-(C44-Pad2): track 58.4 -> 57.4 mm
- net Net-(C39-Pad2): track 52.6 -> 51.6 mm
- net Net-(U10B-+): track 6.32 -> 5.33 mm
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