File: USB_DAC-AMP_V4_credit_card/USB_DAC-AMP_V4_credit_card.kicad_sch (KiCad schematic)
At the start: 121 parts, among them J1 USB_C_Receptacle, J2 SJ-3524-SMT, U1 PCM2900C, U10 NE5532, U11 NE5532, U2 TPS61040DBV, U3 SPX3819M5-L, U4 SPX3819M5-L, U5 NE5532, U6 NE5532, U7 NE5532, U8 NE5532, U9 NE5532, Y3 12 MHz Crystal

Commit message: created V4 to change board dimensions, update schematic
changed out caps to be electrolytic
board dimensions are now whole numbers
Parts:
- added C47: 100n, Capacitor_SMD:C_0603_1608Metric_Pad1.08x0.95mm_HandSolder, symbol Device:C
- added H1, H2, H3, H4: MountingHole, MountingHole:MountingHole_3.5mm, symbol Mechanical:MountingHole
- C1, C10, C11, C12, C13, C19, C9: LCSC (none) -> C1035
- C14, C15, C35, C45: LCSC (none) -> C696799
- C16, C17, C18, C20, C21, C22, C7, C8: LCSC (none) -> C1592
- C2, C23, C24, C3, C33, C36, C4, C43, C46, C5, C6: LCSC (none) -> C1658
- C25, C30, C31, C40, C41: LCSC (none) -> C132558
- C26, C28, C32, C34, C38, C42, C44: LCSC (none) -> C1590
- C27: value 1000u -> 100u; LCSC (none) -> C132558
- C29, C39: LCSC (none) -> C1028
- C37: LCSC (none) -> C1002
- R17: value 2.2 -> 1
- R20, R21: value 1.5k -> 5.1K
- R3: footprint PTN092-H20115K1A:TRIM_PTN092-H20115K1A -> Imported_footprints:TRIM_PTN092-H20115K1A
Connections:
- net +16V: now also FB2.2; no longer FB2.1
- net +16VA: now also FB2.1; no longer FB2.2
- net GND: now also C47.1
- net VBL: no longer R36.2, R39.2
- net VBR: now also R36.2, R39.2
- net VREF: now also C47.2
- net at C41.2: now also R3.2_1; no longer R3.2_2
- net at C43.2, R40.1, U10.7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: now also R3.3_1; no longer R3.3_2
- net at C35.1, R32.1: now also R31.2; no longer R31.1
- net at U8.1, U8.2 (-): now also R26.2; no longer R35.1
- net at C39.2, U8.5 (+): now also R26.1; no longer R35.2
- net at C29.2, U5.5 (+): now also R35.2; no longer R26.2
- net at C33.2, R30.1, U7.3 (+)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: now also R3.3_2, U7.5 (+); no longer R3.3_1, U7.6 (-)
- net at U7.1, U7.2 (-): now also R31.1; no longer R31.2
- net at C31.2: now also R3.2_2; no longer R3.2_1
- net at R32.2, U7.7: now also U7.6 (-); no longer U7.5 (+)
- net at C40.2: now also R3.1_1; no longer R3.1_2
- net at U5.1, U5.2 (-): now also R35.1; no longer R26.1
- net at C30.2: now also R3.1_2; no longer R3.1_1
Other:
- note added: "check this, datasheet says 10uf"
- moved on the sheet: C27, C31, FB2, R26, R31, R35

Commit message: updated V4
Parts:
- removed C14, C15, C35, C45: 1000u, Capacitor_Tantalum_SMD:CP_EIA-7343-43_Kemet-X_HandSolder, symbol Device:C
- removed C25, C27, C30, C31, C40, C41: 100u, Capacitor_Tantalum_SMD:CP_EIA-7343-43_Kemet-X_HandSolder, symbol Device:C
- removed C37: 100u, Capacitor_Tantalum_SMD:CP_EIA-7343-15_Kemet-W, symbol Device:C
- removed C47: 100n, Capacitor_SMD:C_0603_1608Metric_Pad1.08x0.95mm_HandSolder, symbol Device:C
- added C26, C38: 1000u, Capacitor_SMD:CP_Elec_10x10.5, symbol Device:C_Polarized
- added C27, C29, C32, C35, C39, C41, C44, C7: 100u, Capacitor_SMD:CP_Elec_6.3x7.7, symbol Device:C_Polarized
- C1: renamed from C7; footprint Capacitor_SMD:C_0603_1608Metric_Pad1.08x0.95mm_HandSolder -> Capacitor_SMD:C_0603_1608Metric
- C10: renamed from C2; footprint Capacitor_SMD:C_0603_1608Metric_Pad1.08x0.95mm_HandSolder -> Capacitor_SMD:C_0603_1608Metric
- C11: renamed from C17; footprint Capacitor_SMD:C_0603_1608Metric_Pad1.08x0.95mm_HandSolder -> Capacitor_SMD:C_0603_1608Metric
- C12: renamed from C4; footprint Capacitor_SMD:C_0603_1608Metric_Pad1.08x0.95mm_HandSolder -> Capacitor_SMD:C_0603_1608Metric
- C13: renamed from C5; footprint Capacitor_SMD:C_0603_1608Metric_Pad1.08x0.95mm_HandSolder -> Capacitor_SMD:C_0603_1608Metric
- C14: renamed from C16; footprint Capacitor_SMD:C_0603_1608Metric_Pad1.08x0.95mm_HandSolder -> Capacitor_SMD:C_0603_1608Metric
- C15: renamed from C24; footprint Capacitor_SMD:C_0603_1608Metric_Pad1.08x0.95mm_HandSolder -> Capacitor_SMD:C_0603_1608Metric
- C16: renamed from C23; footprint Capacitor_SMD:C_0603_1608Metric_Pad1.08x0.95mm_HandSolder -> Capacitor_SMD:C_0603_1608Metric
- C17: renamed from C10; footprint Capacitor_SMD:C_0603_1608Metric_Pad1.08x0.95mm_HandSolder -> Capacitor_SMD:C_0603_1608Metric
- C18: renamed from C11; footprint Capacitor_SMD:C_0603_1608Metric_Pad1.08x0.95mm_HandSolder -> Capacitor_SMD:C_0603_1608Metric
- C19: renamed from C22; footprint Capacitor_SMD:C_0603_1608Metric_Pad1.08x0.95mm_HandSolder -> Capacitor_SMD:C_0603_1608Metric
- C2: renamed from C8; footprint Capacitor_SMD:C_0603_1608Metric_Pad1.08x0.95mm_HandSolder -> Capacitor_SMD:C_0603_1608Metric
- C20: renamed from C21; footprint Capacitor_SMD:C_0603_1608Metric_Pad1.08x0.95mm_HandSolder -> Capacitor_SMD:C_0603_1608Metric
- C21: renamed from C20; footprint Capacitor_SMD:C_0603_1608Metric_Pad1.08x0.95mm_HandSolder -> Capacitor_SMD:C_0603_1608Metric
- C22: renamed from C19; footprint Capacitor_SMD:C_0603_1608Metric_Pad1.08x0.95mm_HandSolder -> Capacitor_SMD:C_0603_1608Metric
- C23: renamed from C18; footprint Capacitor_SMD:C_0603_1608Metric_Pad1.08x0.95mm_HandSolder -> Capacitor_SMD:C_0603_1608Metric
- C24: renamed from C34; footprint Capacitor_SMD:C_0603_1608Metric_Pad1.08x0.95mm_HandSolder -> Capacitor_SMD:C_0603_1608Metric
- C25: renamed from C28; footprint Capacitor_SMD:C_0603_1608Metric_Pad1.08x0.95mm_HandSolder -> Capacitor_SMD:C_0603_1608Metric
- C28: renamed from C36; footprint Capacitor_SMD:C_0603_1608Metric_Pad1.08x0.95mm_HandSolder -> Capacitor_SMD:C_0603_1608Metric
- C3: renamed from C1; footprint Capacitor_SMD:C_0603_1608Metric_Pad1.08x0.95mm_HandSolder -> Capacitor_SMD:C_0603_1608Metric
- C30: renamed from C29; footprint Capacitor_SMD:C_0603_1608Metric_Pad1.08x0.95mm_HandSolder -> Capacitor_SMD:C_0603_1608Metric
- C31: renamed from C33; footprint Capacitor_SMD:C_0603_1608Metric_Pad1.08x0.95mm_HandSolder -> Capacitor_SMD:C_0603_1608Metric
- C33: renamed from C32; footprint Capacitor_SMD:C_0603_1608Metric_Pad1.08x0.95mm_HandSolder -> Capacitor_SMD:C_0603_1608Metric
- C34: renamed from C26; footprint Capacitor_SMD:C_0603_1608Metric_Pad1.08x0.95mm_HandSolder -> Capacitor_SMD:C_0603_1608Metric
- C36: renamed from C44; footprint Capacitor_SMD:C_0603_1608Metric_Pad1.08x0.95mm_HandSolder -> Capacitor_SMD:C_0603_1608Metric
- C37: renamed from C38; footprint Capacitor_SMD:C_0603_1608Metric_Pad1.08x0.95mm_HandSolder -> Capacitor_SMD:C_0603_1608Metric
- C4: renamed from C6; footprint Capacitor_SMD:C_0603_1608Metric_Pad1.08x0.95mm_HandSolder -> Capacitor_SMD:C_0603_1608Metric
- C40: renamed from C46; footprint Capacitor_SMD:C_0603_1608Metric_Pad1.08x0.95mm_HandSolder -> Capacitor_SMD:C_0603_1608Metric
- C42: renamed from C39; footprint Capacitor_SMD:C_0603_1608Metric_Pad1.08x0.95mm_HandSolder -> Capacitor_SMD:C_0603_1608Metric
- C43: footprint Capacitor_SMD:C_0603_1608Metric_Pad1.08x0.95mm_HandSolder -> Capacitor_SMD:C_0603_1608Metric
- C45: renamed from C42; footprint Capacitor_SMD:C_0603_1608Metric_Pad1.08x0.95mm_HandSolder -> Capacitor_SMD:C_0603_1608Metric
- C5: renamed from C9; footprint Capacitor_SMD:C_0603_1608Metric_Pad1.08x0.95mm_HandSolder -> Capacitor_SMD:C_0603_1608Metric
- C6: renamed from C12; footprint Capacitor_SMD:C_0603_1608Metric_Pad1.08x0.95mm_HandSolder -> Capacitor_SMD:C_0603_1608Metric
- C8: renamed from C13; footprint Capacitor_SMD:C_0603_1608Metric_Pad1.08x0.95mm_HandSolder -> Capacitor_SMD:C_0603_1608Metric
- C9: renamed from C3; footprint Capacitor_SMD:C_0603_1608Metric_Pad1.08x0.95mm_HandSolder -> Capacitor_SMD:C_0603_1608Metric
- D1: renamed from D4; LCSC (none) -> C2480
- D2: renamed from D3; footprint LED_SMD:LED_0603_1608Metric_Pad1.05x0.95mm_HandSolder -> LED_SMD:LED_0603_1608Metric
- D3: renamed from D1; footprint Diode_SMD:D_0603_1608Metric_Pad1.05x0.95mm_HandSolder -> Diode_SMD:D_0603_1608Metric; LCSC (none) -> C316055
- D4: renamed from D2; value 0603ESDA-18N -> D_TVS; footprint Diode_SMD:D_0603_1608Metric_Pad1.05x0.95mm_HandSolder -> Diode_SMD:D_0603_1608Metric
- D5: LCSC (none) -> C2480
- D6, D7: footprint Diode_SMD:D_0603_1608Metric_Pad1.05x0.95mm_HandSolder -> Diode_SMD:D_0603_1608Metric; LCSC (none) -> C316055
- F1: footprint Fuse:Fuse_0603_1608Metric_Pad1.05x0.95mm_HandSolder -> Fuse:Fuse_0603_1608Metric; LCSC (none) -> C20787
- FB1, FB2, FB3, FB4, FB5: footprint Resistor_SMD:R_0603_1608Metric_Pad0.98x0.95mm_HandSolder -> Resistor_SMD:R_0603_1608Metric; LCSC (none) -> C12391
- J1: LCSC (none) -> C5184243
- L1: footprint Inductor_SMD:L_0805_2012Metric_Pad1.05x1.20mm_HandSolder -> Inductor_SMD:L_0805_2012Metric; LCSC (none) -> C223269
- R1: renamed from R12; footprint Resistor_SMD:R_0603_1608Metric_Pad0.98x0.95mm_HandSolder -> Resistor_SMD:R_0603_1608Metric
- R10: renamed from R22; footprint Resistor_SMD:R_0603_1608Metric_Pad0.98x0.95mm_HandSolder -> Resistor_SMD:R_0603_1608Metric
- R11: renamed from R20; footprint Resistor_SMD:R_0603_1608Metric_Pad0.98x0.95mm_HandSolder -> Resistor_SMD:R_0603_1608Metric; LCSC (none) -> C122969
- R12: renamed from R21; footprint Resistor_SMD:R_0603_1608Metric_Pad0.98x0.95mm_HandSolder -> Resistor_SMD:R_0603_1608Metric; LCSC (none) -> C122969
- R13: renamed from R7; footprint Resistor_SMD:R_0603_1608Metric_Pad0.98x0.95mm_HandSolder -> Resistor_SMD:R_0603_1608Metric
- R14: renamed from R8; footprint Resistor_SMD:R_0603_1608Metric_Pad0.98x0.95mm_HandSolder -> Resistor_SMD:R_0603_1608Metric
- R15: renamed from R9; footprint Resistor_SMD:R_0603_1608Metric_Pad0.98x0.95mm_HandSolder -> Resistor_SMD:R_0603_1608Metric
- R16, R36, R39: footprint Resistor_SMD:R_0603_1608Metric_Pad0.98x0.95mm_HandSolder -> Resistor_SMD:R_0603_1608Metric
- R17: renamed from R14; footprint Resistor_SMD:R_0603_1608Metric_Pad0.98x0.95mm_HandSolder -> Resistor_SMD:R_0603_1608Metric
- R18: renamed from R15; footprint Resistor_SMD:R_0603_1608Metric_Pad0.98x0.95mm_HandSolder -> Resistor_SMD:R_0603_1608Metric
- R19: renamed from R31; footprint Resistor_SMD:R_0603_1608Metric_Pad0.98x0.95mm_HandSolder -> Resistor_SMD:R_0603_1608Metric
- R2: renamed from R5; footprint Resistor_SMD:R_0603_1608Metric_Pad0.98x0.95mm_HandSolder -> Resistor_SMD:R_0603_1608Metric
- R20: renamed from R23; footprint Resistor_SMD:R_0603_1608Metric_Pad0.98x0.95mm_HandSolder -> Resistor_SMD:R_0603_1608Metric
- R22: renamed from R35; footprint Resistor_SMD:R_0603_1608Metric_Pad0.98x0.95mm_HandSolder -> Resistor_SMD:R_0603_1608Metric
- R23: renamed from R33; footprint Resistor_SMD:R_0603_1608Metric_Pad0.98x0.95mm_HandSolder -> Resistor_SMD:R_0603_1608Metric
- R24: renamed from R30; footprint Resistor_SMD:R_0603_1608Metric_Pad0.98x0.95mm_HandSolder -> Resistor_SMD:R_0603_1608Metric; LCSC (none) -> C122969
- R25: renamed from R27; footprint Resistor_SMD:R_0603_1608Metric_Pad0.98x0.95mm_HandSolder -> Resistor_SMD:R_0603_1608Metric
- R26: renamed from R28; footprint Resistor_SMD:R_0603_1608Metric_Pad0.98x0.95mm_HandSolder -> Resistor_SMD:R_0603_1608Metric
- R27: renamed from R32; footprint Resistor_SMD:R_0603_1608Metric_Pad0.98x0.95mm_HandSolder -> Resistor_SMD:R_0603_1608Metric
- R28: renamed from R29; footprint Resistor_SMD:R_0603_1608Metric_Pad0.98x0.95mm_HandSolder -> Resistor_SMD:R_0603_1608Metric
- R29: renamed from R24; footprint Resistor_SMD:R_0603_1608Metric_Pad0.98x0.95mm_HandSolder -> Resistor_SMD:R_0603_1608Metric
- R3: renamed from R10; footprint Resistor_SMD:R_0603_1608Metric_Pad0.98x0.95mm_HandSolder -> Resistor_SMD:R_0603_1608Metric
- R30: renamed from R25; footprint Resistor_SMD:R_0603_1608Metric_Pad0.98x0.95mm_HandSolder -> Resistor_SMD:R_0603_1608Metric
- R31: renamed from R41; footprint Resistor_SMD:R_0603_1608Metric_Pad0.98x0.95mm_HandSolder -> Resistor_SMD:R_0603_1608Metric
- R32: renamed from R34; footprint Resistor_SMD:R_0603_1608Metric_Pad0.98x0.95mm_HandSolder -> Resistor_SMD:R_0603_1608Metric
- R33: renamed from R26; footprint Resistor_SMD:R_0603_1608Metric_Pad0.98x0.95mm_HandSolder -> Resistor_SMD:R_0603_1608Metric
- R34: renamed from R43; footprint Resistor_SMD:R_0603_1608Metric_Pad0.98x0.95mm_HandSolder -> Resistor_SMD:R_0603_1608Metric
- R35: renamed from R40; footprint Resistor_SMD:R_0603_1608Metric_Pad0.98x0.95mm_HandSolder -> Resistor_SMD:R_0603_1608Metric; LCSC (none) -> C122969
- R37: renamed from R38; footprint Resistor_SMD:R_0603_1608Metric_Pad0.98x0.95mm_HandSolder -> Resistor_SMD:R_0603_1608Metric
- R38: renamed from R42; footprint Resistor_SMD:R_0603_1608Metric_Pad0.98x0.95mm_HandSolder -> Resistor_SMD:R_0603_1608Metric
- R4: renamed from R13; footprint Resistor_SMD:R_0603_1608Metric_Pad0.98x0.95mm_HandSolder -> Resistor_SMD:R_0603_1608Metric
- R5: renamed from R1; footprint Resistor_SMD:R_0603_1608Metric_Pad0.98x0.95mm_HandSolder -> Resistor_SMD:R_0603_1608Metric; LCSC (none) -> C122969
- R6: renamed from R2; footprint Resistor_SMD:R_0603_1608Metric_Pad0.98x0.95mm_HandSolder -> Resistor_SMD:R_0603_1608Metric; LCSC (none) -> C122969
- R7: renamed from R6; footprint Resistor_SMD:R_0603_1608Metric_Pad0.98x0.95mm_HandSolder -> Resistor_SMD:R_0603_1608Metric
- R8: renamed from R11; footprint Resistor_SMD:R_0603_1608Metric_Pad0.98x0.95mm_HandSolder -> Resistor_SMD:R_0603_1608Metric
- R9: renamed from R17; footprint Resistor_SMD:R_0603_1608Metric_Pad0.98x0.95mm_HandSolder -> Resistor_SMD:R_0603_1608Metric
- U1: renamed from U2; LCSC (none) -> C7722
- U10: renamed from U8; LCSC (none) -> C7426
- U11: renamed from U10; LCSC (none) -> C7426
- U2: renamed from U4; LCSC (none) -> C9056
- U3: LCSC (none) -> C9056
- U4: renamed from U1; LCSC (none) -> C180425
- U5: renamed from U7; LCSC (none) -> C7426
- U6: renamed from U5; LCSC (none) -> C7426
- U7: renamed from U9; LCSC (none) -> C7426
- U8: renamed from U6; LCSC (none) -> C7426
- U9: renamed from U11; LCSC (none) -> C7426
- Y1: renamed from Y3; LCSC (none) -> C9002
- renumbered R3 to R21, TP4 to TP3, TP3 to TP4, TP6 to TP5, TP7 to TP6, TP5 to TP7
Connections:
- net +15VA: now also C7.1
- net GND: now also C35.2, C7.2
- net VOUTL: now also C29.2
- net VOUTR: now also C41.2
- net VREF: now also C35.1
- net at R36.1, U11.3 (+): now also C44.1
- net at R21.2_1: now also C44.2
- net at R19.2, R27.1: now also C26.1
- net at FB4.1, R23.1: now also C26.2
- net at R31.1, R38.1: now also C38.1
- net at U6.6 (-), U6.7: now also C27.1
- net at R32.2, U10.3 (+): now also C41.1
- net at R20.2, U6.3 (+): now also C29.1
- net at R25.1, U7.3 (+): now also C32.1
- net at R21.2_2: now also C32.2
- net at U10.6 (-), U10.7: now also C39.1
- net at R21.1_1: now also C39.2
- net at FB5.1, R34.1: now also C38.2
- net at R21.1_2: now also C27.2
Other:
- note removed: "Chose fairly sizeable electrolytic capacitors, if chosing ceramic, especially in the signal path, chose type cog for bypass, use whatever"
- note removed: "Make sure that the pins in the layout match up and all are accounted for, including voltage lines, check why only A4 is tied to VBUS, cross check with Phil's lab video"
- note removed: "check this, datasheet says 10uf"
- moved on the sheet: C11, C14, C15, C16, C19, C20, C21, C22, C23, C3, C4, C5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

Commit message: Finished V4 layout
Parts:
- added TP11: buffer2_r, TestPoint:TestPoint_Pad_1.0x1.0mm, symbol Connector:TestPoint
- added TP12: buffer2_l, TestPoint:TestPoint_Pad_1.0x1.0mm, symbol Connector:TestPoint
- added TP13: in_l, TestPoint:TestPoint_Pad_1.0x1.0mm, symbol Connector:TestPoint
- added TP14: in_r, TestPoint:TestPoint_Pad_1.0x1.0mm, symbol Connector:TestPoint
- added TP15: buffer1_l, TestPoint:TestPoint_Pad_1.0x1.0mm, symbol Connector:TestPoint
- added TP16: buffer1_r, TestPoint:TestPoint_Pad_1.0x1.0mm, symbol Connector:TestPoint
Connections:
- net at C38.1, R31.1, R38.1: now also TP11.1
- net at C29.1, R20.2, U6.3 (+): now also TP13.1
- net at C41.1, R32.2, U10.3 (+): now also TP14.1
- net at C26.1, R19.2, R27.1: now also TP12.1
- net at C27.2, R21.1_2: now also TP15.1
- net at C39.2, R21.1_1: now also TP16.1
Other:
- moved on the sheet: C26, C27, C29, C38, C39, C41

Commit message: Submitted V1 to Kicad
Parts:
- added R40: 1.5K, Resistor_SMD:R_0603_1608Metric, symbol Device:R
- D2: LCSC (none) -> C84265
- D4: LCSC (none) -> C316055
- R1: LCSC (none) -> C136969
- R10, R2: LCSC (none) -> C326730
- R13, R14, R15, R20, R28, R29, R30, R32, R39, R8: LCSC (none) -> C217885
- R16, R22, R23, R26, R33, R34, R37, R4: LCSC (none) -> C193681
- R17, R18: LCSC (none) -> C217888
- R19, R27, R31, R38, R9: LCSC (none) -> C412388
- R25, R36: value 1.5K -> 22K; LCSC (none) -> C217885
- R3: LCSC (none) -> C217899
- R7: LCSC (none) -> C705797
- U10, U11, U5, U6, U7, U8, U9: footprint Package_SO:SOIC-8_5.3x5.3mm_P1.27mm -> Package_SO:SOIC-8_3.9x4.9mm_P1.27mm
Connections:
- net VDDI: now also R40.1
- net at U4.28 (~{SSPND}): now also R40.2
- no-connect marks 17 -> 16
